File: hw/ControllerBoard/ControllerBoard.sch (KiCad schematic (older format))
At the start: 29 parts, among them J1 Screw_Terminal_01x02, Q1 2N3906, Q2 2N3906, Q3 2N3906, Q4 2N3906, SW1 SW_Push, SW2 SW_Push, SW3 SW_Push, U1 DS1307+, Y1 32.768 KHz

Commit message: updated schematic for controller board
Parts:
- removed AFF1, AFF2, AFF3, AFF4: LTS-6960HR, Display_7Segment:7SegmentLED_LTS6760_LTS6780, symbol Display_Character:LTS-6960HR
- removed Q1, Q2, Q3, Q4: 2N3906, symbol device:Q_PNP_EBC
- removed R1, R2, R3, R4, R5, R6, R7, R8: R, symbol device:R
- removed R12, R13, R14, R9: 4k7, symbol device:R
- removed SW1, SW2, SW3: SW_Push, symbol Switch:SW_Push
- added J2: Conn_01x06_Male, symbol Connector:Conn_01x06_Male
- added J3: Conn_02x08_Odd_Even, symbol Connector_Generic:Conn_02x08_Odd_Even
- R1: renamed from R10; value 1k -> 1k5
- R2: renamed from R11; value 1k -> 1k5
Connections:
- wire segments 156 -> 92
Other:
- note added: "Connector for ribbon cable\nto display board"
- note added: "Connector for set/hour/minute\npush buttons"
- note added: "Hex clock controller board"
- note removed: "Hex clock using Arduino Nano and DS1307 RTC"
- moved on the sheet: J1, R1, R2, TB1, U1, Y1

Commit message: annotated with component footprints
Parts:
- J1: footprint (none) -> TerminalBlock_Phoenix:TerminalBlock_Phoenix_MKDS-1,5-2_1x02_P5.00mm_Horizontal
- J2: footprint (none) -> Pin_Headers:Pin_Header_Straight_1x06_Pitch2.54mm
- J3: footprint (none) -> Pin_Headers:Pin_Header_Straight_2x08_Pitch2.54mm
- R1, R2: footprint (none) -> Resistors_ThroughHole:R_Axial_DIN0207_L6.3mm_D2.5mm_P7.62mm_Horizontal
- TB1: footprint SHIELD_ARDUINO_NANO -> ARDUINO_NANO:SHIELD_ARDUINO_NANO
- Y1: footprint (none) -> AB26TRB-32.768KHZ-T:XTAL_AB26TRB-32.768KHZ-T
Changed lines of the file:
@@
 F 0 "Y1" V 4854 5931 50  0000 L CNN
 F 1 "32.768 KHz" V 4945 5931 50  0000 L CNN
-F 2 "" H 4900 5800 50  0001 C CNN
+F 2 "AB26TRB-32.768KHZ-T:XTAL_AB26TRB-32.768KHZ-T" H 4900 5800 50  0001 C CNN
 F 3 "" H 4900 5800 50  0001 C CNN
 	1    4900 5800
@@
 F 0 "R1" H 5030 4996 50  0000 R CNN
 F 1 "1k5" H 5030 4905 50  0000 R CNN
-F 2 "" V 5030 4950 50  0001 C CNN
+F 2 "Resistors_ThroughHole:R_Axial_DIN0207_L6.3mm_D2.5mm_P7.62mm_Horizontal" V 5030 4950 50  0001 C CNN
 F 3 "" H 5100 4950 50  0001 C CNN
 	1    5100 4950
@@
 F 0 "R2" H 5330 4996 50  0000 R CNN
 F 1 "1k5" H 5330 4905 50  0000 R CNN
-F 2 "" V 5330 4950 50  0001 C CNN
+F 2 "Resistors_ThroughHole:R_Axial_DIN0207_L6.3mm_D2.5mm_P7.62mm_Horizontal" V 5330 4950 50  0001 C CNN
 F 3 "" H 5400 4950 50  0001 C CNN
 	1    5400 4950
@@
 F 0 "J1" H 7730 2942 50  0000 L CNN
 F 1 "Screw_Terminal_01x02" H 7730 2851 50  0000 L CNN
-F 2 "" H 7650 2950 50  0001 C CNN
+F 2 "TerminalBlock_Phoenix:TerminalBlock_Phoenix_MKDS-1,5-2_1x02_P5.00mm_Horizontal" H 7650 2950 50  0001 C CNN
 F 3 "~" H 7650 2950 50  0001 C CNN
 	1    7650 2950
@@
 F 0 "TB1" H 3250 5467 50  0000 C CNN
 F 1 "ARDUINO_NANO" H 3250 5376 50  0000 C CNN
-F 2 "SHIELD_ARDUINO_NANO" H 3250 3900 50  0001 L BNN
+F 2 "ARDUINO_NANO:SHIELD_ARDUINO_NANO" H 3250 3900 50  0001 L BNN
 F 3 "DFRobot" H 3250 3900 50  0001 L BNN
 F 4 "Dev.kit: Arduino; UART; ICSP, USB B mini, pin strips" H 3250 3900 50  0001 L BNN "Field4"
@@
 F 0 "J2" H 6073 3130 50  0000 R CNN
 F 1 "Conn_01x06_Male" H 6073 3221 50  0000 R CNN
-F 2 "" H 6100 3250 50  0001 C CNN
+F 2 "Pin_Headers:Pin_Header_Straight_1x06_Pitch2.54mm" H 6100 3250 50  0001 C CNN
 F 3 "~" H 6100 3250 50  0001 C CNN
 	1    6100 3250
@@
 F 0 "J3" H 8200 5617 50  0000 C CNN
 F 1 "Conn_02x08_Odd_Even" H 8200 5526 50  0000 C CNN
-F 2 "" H 8150 5100 50  0001 C CNN
+F 2 "Pin_Headers:Pin_Header_Straight_2x08_Pitch2.54mm" H 8150 5100 50  0001 C CNN
 F 3 "~" H 8150 5100 50  0001 C CNN
 	1    8150 5100

Commit message: fix some footprints, start PCB
Parts:
- U1: footprint Package_DIP:DIP-8_W7.62mm -> Housings_DIP:DIP-8_W7.62mm_Socket
- Y1: footprint AB26TRB-32.768KHZ-T:XTAL_AB26TRB-32.768KHZ-T -> Crystals:Crystal_C38-LF_d3.0mm_l8.0mm_Horizontal
Changed lines of the file:
@@
 F 0 "U1" H 6591 5496 50  0000 L CNN
 F 1 "DS1307+" H 6591 5405 50  0000 L CNN
-F 2 "Package_DIP:DIP-8_W7.62mm" H 6050 4950 50  0001 C CNN
+F 2 "Housings_DIP:DIP-8_W7.62mm_Socket" H 6050 4950 50  0001 C CNN
 F 3 "https://datasheets.maximintegrated.com/en/ds/DS1307.pdf" H 6050 5250 50  0001 C CNN
 	1    6050 5450
@@
 F 0 "Y1" V 4854 5931 50  0000 L CNN
 F 1 "32.768 KHz" V 4945 5931 50  0000 L CNN
-F 2 "AB26TRB-32.768KHZ-T:XTAL_AB26TRB-32.768KHZ-T" H 4900 5800 50  0001 C CNN
+F 2 "Crystals:Crystal_C38-LF_d3.0mm_l8.0mm_Horizontal" H 4900 5800 50  0001 C CNN
 F 3 "" H 4900 5800 50  0001 C CNN
 	1    4900 5800
