File: hw/ControllerBoard/ControllerBoard.kicad_pcb (KiCad board)
At the start: 2 copper layers, 71.1 x 50.8 mm, 12 parts, among them J1 Screw_Terminal_01x02, J2 Conn_01x06_Male, J3 Conn_02x08_Odd_Even, U1 DS1307+, Y1 32.768 KHz

Commit message: routed all nets, board is ready?
Parts:
- moved R2 14.4 mm to (81.8, 88.4), turned to 180 degrees
- moved J2 11.7 mm to (107.2, 67.6), turned to 180 degrees
- moved R1 11.4 mm to (81.8, 85.1), turned to 180 degrees
- moved TB1 2.54 mm to (73.4, 73.4)
- moved Y1 1.83 mm to (99.8, 84.1)
- moved J1 0.92 mm to (116.1, 90.9)
- moved U1 0.51 mm to (99.8, 80.8)
Routing:
- net VCC: track 0.00 -> 145.1 mm
- net GND: track 0.00 -> 101.1 mm
- net /SW1: track 0.00 -> 58.3 mm
- net /SW3: track 0.00 -> 50.6 mm, vias 0 -> 1
- net /SW2: track 0.00 -> 50.1 mm
- net /SDA: track 0.00 -> 47.4 mm
- net /SCL: track 0.00 -> 37.0 mm
- net /D0: track 0.00 -> 36.3 mm
- net /D1: track 0.00 -> 35.4 mm
- net /D2: track 0.00 -> 25.0 mm, vias 0 -> 1
- net /AN3: track 0.00 -> 23.3 mm
- net /AN2: track 0.00 -> 21.0 mm
- net /D3: track 0.00 -> 20.2 mm, vias 0 -> 1
- net /D7: track 0.00 -> 17.4 mm
- net /AN0: track 0.00 -> 15.9 mm, vias 0 -> 1
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- added copper zone on B.Cu, net GND
- added copper zone on F.Cu, net VCC
Other:
- net class Default: clearance 0.2 -> 0.1524; trace_width 0.25 -> 0.1524; via_dia 0.8 -> 0.6858; via_drill 0.4 -> 0.3302
- rule trace_clearance: 0.2 -> 0.1524
- rule trace_min: 0.2 -> 0.1524
- rule via_min_drill: 0.3 -> 0.254
- rule via_min_size: 0.4 -> 0.508
- board text added: "+5V"
- board text added: "GND"
- board text added: "HexClock controller board 0.1 11-May-2019 https://github.com/daveho/HexClock"
- board text added: "SW1"
- board text added: "SW2"
- board text added: "SW3"
